File: keyboard_macropad/keyboard_macropad/keyboard_macropad.kicad_pcb (KiCad board)
At the start: 2 copper layers, 88 x 131 mm, 42 parts, among them J1 Conn_01x04_Pin, J2 Conn_01x04_Pin, J3 Conn_01x04_Pin, J4 Conn_01x04_Pin, SW1 SW_Push, SW10 SW_Push, SW11 SW_Push, SW12 SW_Push, SW13 SW_Push, SW14 SW_Push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

Commit message: updates
Parts:
- SW1, SW10, SW11, SW12, SW13, SW14, SW15, SW16, SW2, SW3, SW4, SW5, SW6, SW7, SW8, SW9: footprint Button_Switch_Keyboard:SW_Cherry_MX_1.00u_PCB -> dakshmessesaround:jiggupiggu
Other:
- outline, holes or cut-outs redrawn
